Commit message: somthing is wong'

File: kene_robot/urdf/robot.xacro (robot description, xacro)
@@ -1,5 +1,5 @@
 <?xml version='1.0'?>
 <robot name="robot" xmlns:xacro="http://www.ros.org/wiki/xacro">
-	<xacro:include filename="$(find go_chase_it)/urdf/robot.gazebo"/>
+	<xacro:include filename="$(find kene_robot)/urdf/robot.gazebo"/>
 	<link name="robot_footprint"></link>
 	<joint name="robot_footprint_joint" type="fixed">
@@ -165,5 +165,5 @@
 			<origin xyz="0 0 0" rpy=" 0 0 0"/>
 			<geometry>
-				<mesh filename="package://go_chase_it/meshes/hokuyo.dae"/>
+				<mesh filename="package://kene_robot/meshes/hokuyo.dae"/>
 			</geometry>
 		</visual>

Commit message: adding RGB-d

File: kene_robot/urdf/robot.xacro (robot description, xacro)
@@ -175,4 +175,12 @@
 		<axis xyz="0 1 0" rpy="0 0 0"/>
 	</joint>
+	<!--RGB-D -->
+	<joint name="camera_optical_joint" type="fixed">
+		<origin xyz="0 0 0" rpy="-1.5707 0 -1.5707"/>
+		<parent link="camera_link"/>
+		<child link="camera_link_optical"/>
+	</joint>
+	<link name="camera_link_optical">
+	</link>
 	<gazebo reference="chassis">
 		<material>Gazebo/Green</material>

Commit message: adding teleops

File: kene_robot/urdf/robot.xacro (robot description, xacro)
@@ -178,5 +178,5 @@
 	<joint name="camera_optical_joint" type="fixed">
 		<origin xyz="0 0 0" rpy="-1.5707 0 -1.5707"/>
-		<parent link="camera_link"/>
+		<parent link="camera"/>
 		<child link="camera_link_optical"/>
 	</joint>

Commit message: fixing robot and world

File: kene_robot/urdf/robot.xacro (robot description, xacro)
@@ -79,5 +79,5 @@
 	</link>
 	<joint type="continuous" name="left_wheel_hinge">
-		<origin xyz="0 0.125 0" rpy="0 0 0"/>
+		<origin xyz="0 0.15 0" rpy="0 0 0"/>
 		<child link="left_wheel"/>
 		<parent link="chassis"/>
@@ -110,5 +110,5 @@
 	</link>
 	<joint type="continuous" name="right_wheel_hinge">
-		<origin xyz="0 -0.125 0" rpy="0 0 0"/>
+		<origin xyz="0 -0.15 0" rpy="0 0 0"/>
 		<child link="right_wheel"/>
 		<parent link="chassis"/>
@@ -145,9 +145,11 @@
 		<parent link="chassis"/>
 		<axis xyz="0 1 0" rpy="0 0 0"/>
+		<limit effort="10000" velocity="1000"/>
+		<dynamics damping="1.0" friction="1.0"/>
 	</joint>
 	<!--Hokuyo Lidar sensor-->
 	<link name="hokuyo">
 		<inertial>
-			<mass value="1e-5"/>
+			<mass value="0.1"/>
 			<origin xyz="0 0 0" rpy=" 0 0 0"/>
 			<inertia
@@ -159,5 +161,5 @@
 			<origin xyz="0 0 0" rpy=" 0 0 0"/>
 			<geometry>
-				<box size=".1 .1 .1"/>
+				<box size="0.1 0.1 0.1"/>
 			</geometry>
 		</collision>
@@ -174,4 +176,6 @@
 		<parent link="chassis"/>
 		<axis xyz="0 1 0" rpy="0 0 0"/>
+		<limit effort="10000" velocity="1000"/>
+		<dynamics damping="1.0" friction="1.0"/>
 	</joint>
 	<!--RGB-D -->
